File: hw/Watch/MainBoard/Zdroj.kicad_sch (KiCad schematic)
At the start: 22 parts, among them Q1 Q_PMOS_DGS-L, SW4 ON, U2 SL8261D-G3JE

Commit message: wip
Parts:
- SW4: footprint RLK-ElectorMechanicalComponents:TCF2QR -> Button_Switch_SMD:SW_Push_1P1T_NO_Vertical_Wuerth_434133025816; LCSC C240292 -> C127488
Changed lines of the file:
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@@
       (effects (font (size 1.27 1.27)) (justify right))
     )
-    (property "Footprint" "RLK-ElectorMechanicalComponents:TCF2QR" (at 111.76 133.35 0)
+    (property "Footprint" "Button_Switch_SMD:SW_Push_1P1T_NO_Vertical_Wuerth_434133025816" (at 111.76 133.35 0)
       (effects (font (size 1.27 1.27)) hide)
     )
@@
       (effects (font (size 1.27 1.27)) hide)
     )
-    (property "LCSC" "C240292" (at 116.84 133.35 0)
+    (property "LCSC" "C127488" (at 116.84 133.35 0)
       (effects (font (size 1.27 1.27)) hide)
     )
