File: hw/Watch/MainBoard/ESP32-S3-MINI.kicad_sch (KiCad schematic)
At the start: 12 parts, among them J1 ESP-Programing_conector, SW2 EN, SW3 BOOT, U1 ESP32-S3-MINI

Commit message: wip
Parts:
- SW2, SW3: footprint RLK-ElectorMechanicalComponents:TCF2QR -> Button_Switch_SMD:SW_Push_1P1T_NO_Vertical_Wuerth_434133025816; LCSC C240292 -> C127488
Changed lines of the file:
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@@
       (effects (font (size 1.27 1.27)) (justify right))
     )
-    (property "Footprint" "RLK-ElectorMechanicalComponents:TCF2QR" (at 185.42 129.54 0)
+    (property "Footprint" "Button_Switch_SMD:SW_Push_1P1T_NO_Vertical_Wuerth_434133025816" (at 185.42 129.54 0)
       (effects (font (size 1.27 1.27)) hide)
     )
@@
       (effects (font (size 1.27 1.27)) hide)
     )
-    (property "LCSC" "C240292" (at 190.5 129.54 0)
+    (property "LCSC" "C127488" (at 190.5 129.54 0)
       (effects (font (size 1.27 1.27)) hide)
     )
@@
       (effects (font (size 1.27 1.27)) (justify right))
     )
-    (property "Footprint" "RLK-ElectorMechanicalComponents:TCF2QR" (at 172.72 129.54 0)
+    (property "Footprint" "Button_Switch_SMD:SW_Push_1P1T_NO_Vertical_Wuerth_434133025816" (at 172.72 129.54 0)
       (effects (font (size 1.27 1.27)) hide)
     )
@@
       (effects (font (size 1.27 1.27)) hide)
     )
-    (property "LCSC" "C240292" (at 177.8 129.54 0)
-      (effects (font (size 1.27 1.27)) hide)
-    )
+    (property "LCSC" "C127488" (at 177.8 129.54 0)
+      (effects (font (size 1.27 1.27)) hide)
+    )

Commit message: wip
Parts:
- C1: footprint Capacitor_SMD:C_0603_1608Metric -> Capacitor_SMD:C_0402_1005Metric; Basic/Extended B -> E; LCSC C96446 -> C315248; info 25V, X5R -> 10V, X5R
- C2: footprint Capacitor_SMD:C_0402_1005Metric -> Capacitor_SMD:C_0201_0603Metric; Basic/Extended B -> E; LCSC C307331 -> C5142565; info 50V, X7R -> 10V, X5R
- C3, C4: footprint Capacitor_SMD:C_0402_1005Metric -> Capacitor_SMD:C_0201_0603Metric; JLCPCB_CORRECTION 0;0;0 -> (none); LCSC C1518208 -> C76935; info 50V, X5R (potenciálně C52923 což je 25V, X5R ) -> 10V, X5R
- R6, R7, R8, R9: footprint Resistor_SMD:R_0402_1005Metric -> Resistor_SMD:R_0201_0603Metric; Basic/Extended B -> E; JLCPCB_CORRECTION 0;0;0 -> (none); LCSC C25744 -> C106225
- U1: Basic/Extended (none) -> E; LCSC (none) -> C3013941
Connections:
- net IO00-PU renamed BOOT
- net IO03-FLOATING: no longer names the net of U1.7 (IO03-FLOATING)
- net IO45-PD: no longer names the net of R9.1, U1.41 (IO45-PD)
- net IO46-PD: no longer names the net of R8.1, U1.44 (IO46-PD)
- no-connect marks 1 -> 2

Commit message: PCB
Parts:
- C2: footprint Capacitor_SMD:C_0201_0603Metric -> Capacitor_SMD:C_0402_1005Metric; Basic/Extended E -> B; LCSC C5142565 -> C307331; info 10V, X5R -> 50V, X7R
- C3, C4: footprint Capacitor_SMD:C_0201_0603Metric -> Capacitor_SMD:C_0402_1005Metric; Basic/Extended E -> B; LCSC C76935 -> C52923; info 10V, X5R -> 25V, X5R
- R6, R7, R8, R9: footprint Resistor_SMD:R_0201_0603Metric -> Resistor_SMD:R_0402_1005Metric; Basic/Extended E -> B; LCSC C106225 -> C25744
Changed lines of the file:
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@@
       (effects (font (size 1.27 1.27)) (justify right))
     )
-    (property "Footprint" "Capacitor_SMD:C_0201_0603Metric" (at 179.3748 104.14 0)
+    (property "Footprint" "Capacitor_SMD:C_0402_1005Metric" (at 179.3748 104.14 0)
       (effects (font (size 1.27 1.27)) hide)
     )
@@
       (effects (font (size 1.27 1.27)) hide)
     )
-    (property "LCSC" "C76935" (at 180.34 100.33 0)
+    (property "LCSC" "C52923" (at 180.34 100.33 0)
       (effects (font (size 1.27 1.27)) hide)
     )
@@
       (effects (font (size 1.27 1.27)) hide)
     )
-    (property "Basic/Extended" "E" (at 180.34 100.33 0)
-      (effects (font (size 1.27 1.27)) hide)
-    )
-    (property "info" "10V, X5R" (at 180.34 100.33 0)
+    (property "Basic/Extended" "B" (at 180.34 100.33 0)
+      (effects (font (size 1.27 1.27)) hide)
+    )
+    (property "info" "25V, X5R" (at 180.34 100.33 0)
       (effects (font (size 1.27 1.27)) hide)
     )
@@
       (effects (font (size 1.27 1.27)) (justify left))
     )
-    (property "Footprint" "Resistor_SMD:R_0201_0603Metric" (at 168.402 100.33 90)
+    (property "Footprint" "Resistor_SMD:R_0402_1005Metric" (at 168.402 100.33 90)
       (effects (font (size 1.27 1.27)) hide)
     )
@@
       (effects (font (size 1.27 1.27)) hide)
     )
-    (property "LCSC" "C106225" (at 170.18 100.33 0)
+    (property "LCSC" "C25744" (at 170.18 100.33 0)
       (effects (font (size 1.27 1.27)) hide)
     )
@@
       (effects (font (size 1.27 1.27)) hide)
     )
-    (property "Basic/Extended" "E" (at 170.18 100.33 0)
+    (property "Basic/Extended" "B" (at 170.18 100.33 0)
       (effects (font (size 1.27 1.27)) hide)
     )
@@
       (effects (font (size 1.27 1.27)) (justify left))
     )
-    (property "Footprint" "Resistor_SMD:R_0201_0603Metric" (at 188.722 62.23 90)
+    (property "Footprint" "Resistor_SMD:R_0402_1005Metric" (at 188.722 62.23 90)
       (effects (font (size 1.27 1.27)) hide)
     )
@@
       (effects (font (size 1.27 1.27)) hide)
     )
-    (property "LCSC" "C106225" (at 190.5 62.23 0)
+    (property "LCSC" "C25744" (at 190.5 62.23 0)
       (effects (font (size 1.27 1.27)) hide)
     )
@@
       (effects (font (size 1.27 1.27)) hide)
     )
-    (property "Basic/Extended" "E" (at 190.5 62.23 0)
+    (property "Basic/Extended" "B" (at 190.5 62.23 0)
       (effects (font (size 1.27 1.27)) hide)
     )
@@
       (effects (font (size 1.27 1.27)))
     )
-    (property "Footprint" "Capacitor_SMD:C_0201_0603Metric" (at 224.79 53.0352 0)
+    (property "Footprint" "Capacitor_SMD:C_0402_1005Metric" (at 224.79 53.0352 0)
       (effects (font (size 1.27 1.27)) hide)
     )
@@
       (effects (font (size 1.27 1.27)) hide)
     )
-    (property "LCSC" "C5142565" (at 228.6 52.07 0)
+    (property "LCSC" "C307331" (at 228.6 52.07 0)
       (effects (font (size 1.27 1.27)) hide)
     )
@@
       (effects (font (size 1.27 1.27)) hide)
     )
-    (property "Basic/Extended" "E" (at 228.6 52.07 0)
-      (effects (font (size 1.27 1.27)) hide)
-    )
-    (property "info" "10V, X5R" (at 228.6 52.07 0)
+    (property "Basic/Extended" "B" (at 228.6 52.07 0)
+      (effects (font (size 1.27 1.27)) hide)
+    )
+    (property "info" "50V, X7R" (at 228.6 52.07 0)
       (effects (font (size 1.27 1.27)) hide)
     )
@@
       (effects (font (size 1.27 1.27)) (justify left))
     )
-    (property "Footprint" "Resistor_SMD:R_0201_0603Metric" (at 178.562 76.2 90)
+    (property "Footprint" "Resistor_SMD:R_0402_1005Metric" (at 178.562 76.2 90)
       (effects (font (size 1.27 1.27)) hide)
     )
@@
       (effects (font (size 1.27 1.27)) hide)
     )
-    (property "LCSC" "C106225" (at 180.34 76.2 0)
+    (property "LCSC" "C25744" (at 180.34 76.2 0)
       (effects (font (size 1.27 1.27)) hide)
     )
@@
       (effects (font (size 1.27 1.27)) hide)
     )
-    (property "Basic/Extended" "E" (at 180.34 76.2 0)
+    (property "Basic/Extended" "B" (at 180.34 76.2 0)
       (effects (font (size 1.27 1.27)) hide)
     )
@@
       (effects (font (size 1.27 1.27)) (justify left))
     )
-    (property "Footprint" "Resistor_SMD:R_0201_0603Metric" (at 160.782 100.33 90)
+    (property "Footprint" "Resistor_SMD:R_0402_1005Metric" (at 160.782 100.33 90)
       (effects (font (size 1.27 1.27)) hide)
     )
@@
       (effects (font (size 1.27 1.27)) hide)
     )
-    (property "LCSC" "C106225" (at 162.56 100.33 0)
+    (property "LCSC" "C25744" (at 162.56 100.33 0)
       (effects (font (size 1.27 1.27)) hide)
     )
@@
       (effects (font (size 1.27 1.27)) hide)
     )
-    (property "Basic/Extended" "E" (at 162.56 100.33 0)
+    (property "Basic/Extended" "B" (at 162.56 100.33 0)
       (effects (font (size 1.27 1.27)) hide)
     )
@@
       (effects (font (size 1.27 1.27)) (justify right))
     )
-    (property "Footprint" "Capacitor_SMD:C_0201_0603Metric" (at 189.5348 104.14 0)
+    (property "Footprint" "Capacitor_SMD:C_0402_1005Metric" (at 189.5348 104.14 0)
       (effects (font (size 1.27 1.27)) hide)
     )
@@
       (effects (font (size 1.27 1.27)) hide)
     )
-    (property "LCSC" "C76935" (at 190.5 100.33 0)
+    (property "LCSC" "C52923" (at 190.5 100.33 0)
       (effects (font (size 1.27 1.27)) hide)
     )
@@
       (effects (font (size 1.27 1.27)) hide)
     )
-    (property "Basic/Extended" "E" (at 190.5 100.33 0)
-      (effects (font (size 1.27 1.27)) hide)
-    )
-    (property "info" "10V, X5R" (at 190.5 100.33 0)
-      (effects (font (size 1.27 1.27)) hide)
-    )
+    (property "Basic/Extended" "B" (at 190.5 100.33 0)
+      (effects (font (size 1.27 1.27)) hide)
+    )
+    (property "info" "25V, X5R" (at 190.5 100.33 0)
+      (effects (font (size 1.27 1.27)) hide)
+    )
