File: hw/Watch/MainBoard/LDC.kicad_sch (KiCad schematic)
At the start: 3 parts, among them U3 LDC1x12

Commit message: wip
Parts:
- C5: footprint Capacitor_SMD:C_0402_1005Metric -> Capacitor_SMD:C_0201_0603Metric; JLCPCB_CORRECTION 0;0;0 -> (none); LCSC C1518208 -> C76935; info 50V, X5R (potenciálně C52923 což je 25V, X5R ) -> 10V, X5R
- C6: footprint Capacitor_SMD:C_0402_1005Metric -> Capacitor_SMD:C_0201_0603Metric; Basic/Extended B -> E; LCSC C307331 -> C5142565; info 50V, X7R -> 10V, X5R
- U3: Basic/Extended (none) -> E; LCSC (none) -> C202191
Changed lines of the file:
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@@
+      (effects (font (size 1.27 1.27)) hide)
+    )
+    (property "Basic/Extended" "E" (at 152.4 76.2 0)
+      (effects (font (size 1.27 1.27)) hide)
+    )
+    (property "LCSC" "C202191" (at 152.4 76.2 0)
       (effects (font (size 1.27 1.27)) hide)
     )
@@
       (effects (font (size 1.27 1.27)) (justify left))
     )
-    (property "Footprint" "Capacitor_SMD:C_0402_1005Metric" (at 115.2652 86.36 0)
+    (property "Footprint" "Capacitor_SMD:C_0201_0603Metric" (at 115.2652 86.36 0)
       (effects (font (size 1.27 1.27)) hide)
     )
@@
       (effects (font (size 1.27 1.27)) hide)
     )
-    (property "LCSC" "C307331" (at 114.3 82.55 0)
+    (property "LCSC" "C5142565" (at 114.3 82.55 0)
       (effects (font (size 1.27 1.27)) hide)
     )
-    (property "info" "50V, X7R" (at 114.3 82.55 0)
+    (property "info" "10V, X5R" (at 114.3 82.55 0)
       (effects (font (size 1.27 1.27)) hide)
     )
-    (property "Basic/Extended" "B" (at 114.3 82.55 0)
+    (property "Basic/Extended" "E" (at 114.3 82.55 0)
       (effects (font (size 1.27 1.27)) hide)
     )
@@
       (effects (font (size 1.27 1.27)) (justify left))
     )
-    (property "Footprint" "Capacitor_SMD:C_0402_1005Metric" (at 102.5652 86.36 0)
+    (property "Footprint" "Capacitor_SMD:C_0201_0603Metric" (at 102.5652 86.36 0)
       (effects (font (size 1.27 1.27)) hide)
     )
@@
       (effects (font (size 1.27 1.27)) hide)
     )
-    (property "LCSC" "C1518208" (at 101.6 82.55 0)
+    (property "LCSC" "C76935" (at 101.6 82.55 0)
       (effects (font (size 1.27 1.27)) hide)
     )
-    (property "info" "50V, X5R (potenciálně C52923 což je 25V, X5R )" (at 101.6 82.55 0)
+    (property "info" "10V, X5R" (at 101.6 82.55 0)
       (effects (font (size 1.27 1.27)) hide)
     )
@@
       (effects (font (size 1.27 1.27)) hide)
     )
-    (property "JLCPCB_CORRECTION" "0;0;0" (at 101.6 82.55 0)
+    (property "JLCPCB_CORRECTION" "" (at 101.6 82.55 0)
       (effects (font (size 1.27 1.27)) hide)
     )

Commit message: PCB
Parts:
- C5: footprint Capacitor_SMD:C_0201_0603Metric -> Capacitor_SMD:C_0402_1005Metric; Basic/Extended E -> B; LCSC C76935 -> C52923; info 10V, X5R -> 25V, X5R
- C6: footprint Capacitor_SMD:C_0201_0603Metric -> Capacitor_SMD:C_0402_1005Metric; Basic/Extended E -> B; LCSC C5142565 -> C307331; info 10V, X5R -> 50V, X7R
Changed lines of the file:
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@@
       (effects (font (size 1.27 1.27)) (justify left))
     )
-    (property "Footprint" "Capacitor_SMD:C_0201_0603Metric" (at 115.2652 86.36 0)
+    (property "Footprint" "Capacitor_SMD:C_0402_1005Metric" (at 115.2652 86.36 0)
       (effects (font (size 1.27 1.27)) hide)
     )
@@
       (effects (font (size 1.27 1.27)) hide)
     )
-    (property "LCSC" "C5142565" (at 114.3 82.55 0)
+    (property "LCSC" "C307331" (at 114.3 82.55 0)
       (effects (font (size 1.27 1.27)) hide)
     )
-    (property "info" "10V, X5R" (at 114.3 82.55 0)
+    (property "info" "50V, X7R" (at 114.3 82.55 0)
       (effects (font (size 1.27 1.27)) hide)
     )
-    (property "Basic/Extended" "E" (at 114.3 82.55 0)
+    (property "Basic/Extended" "B" (at 114.3 82.55 0)
       (effects (font (size 1.27 1.27)) hide)
     )
@@
       (effects (font (size 1.27 1.27)) (justify left))
     )
-    (property "Footprint" "Capacitor_SMD:C_0201_0603Metric" (at 102.5652 86.36 0)
+    (property "Footprint" "Capacitor_SMD:C_0402_1005Metric" (at 102.5652 86.36 0)
       (effects (font (size 1.27 1.27)) hide)
     )
@@
       (effects (font (size 1.27 1.27)) hide)
     )
-    (property "LCSC" "C76935" (at 101.6 82.55 0)
+    (property "LCSC" "C52923" (at 101.6 82.55 0)
       (effects (font (size 1.27 1.27)) hide)
     )
-    (property "info" "10V, X5R" (at 101.6 82.55 0)
+    (property "info" "25V, X5R" (at 101.6 82.55 0)
       (effects (font (size 1.27 1.27)) hide)
     )
-    (property "Basic/Extended" "E" (at 101.6 82.55 0)
+    (property "Basic/Extended" "B" (at 101.6 82.55 0)
       (effects (font (size 1.27 1.27)) hide)
     )
