File: hw/Watch/MainBoard/PowerSource.kicad_sch (KiCad schematic)
At the start: 22 parts, among them Q1 Q_PMOS_DGS-L, SW4 ON, U2 SL8261D-G3JE

Commit message: WIP
Parts:
- removed BT1: Battery_Cell, symbol Device:Battery_Cell
- removed Q? (x3): Q_NMOS_DGS-P, Package_SON:Diodes_PowerDI3333-8, symbol RKL-Uncategorized:Si7112DN
- removed TP6: TestPoint-EN_ALL, Connector_Pin:Pin_D0.9mm_L10.0mm_W2.4mm_FlatFork, symbol Connector:TestPoint
- added J2: Conn_01x02, Connector_JST:JST_PH_S2B-PH-SM4-TB_1x02-1MP_P2.00mm_Horizontal, symbol Connector_Generic:Conn_01x02
- added Q2, Q7: PMOS-2x_BSS84DW, RKL-StandardPackages:DFN3030, symbol RKL-Uncategorized:PMOS-2x_BSS84DW
- added Q?: Q_NMOS_DGS-L, Package_TO_SOT_SMD:SOT-23, symbol Device:Q_NMOS_DGS
- added R25: 10k, Resistor_SMD:R_0402_1005Metric, symbol Device:R
- Q? (x2): LCSC C10487 -> C8545
Connections:
- net GND: now also Q7.S2 (S), Q?.3 (S), R25.1; no longer SW4.1
- net VCC: now also SW4.2, J2.2 (Pin_2), Q2.G1 (G), Q2.G2 (G)
- net at C7.2, R13.1, U2.6 (GND): now also Q2.S1 (S), Q2.S2 (S), Q7.S1 (S)
- net at U2.3 (OC): now also Q7.G2 (G)
- net at U2.1 (OD): now also Q7.G1 (G)
- net at C8.2, R15.2: now also Q?.1 (D); no longer Q?.2 (G), SW4.2
- new net: J2.1 (Pin_1), Q2.D1 (D), Q2.D2 (D)
- new net: Q7.D1 (D), Q7.D2 (D)
- new net: Q?.2 (G), Q?.2 (G), R25.2, SW4.1
Other:
- moved on the sheet: C7, C8, C9, Q1, Q?, R10, R11, R13, R14, R15, R16, R17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

Commit message: wip
Parts:
- C7: footprint Capacitor_SMD:C_0402_1005Metric -> Capacitor_SMD:C_0201_0603Metric; Basic/Extended B -> E; LCSC C307331 -> C5142565; info 50V, X7R -> 10V, X5R
- C8, C9: footprint Capacitor_SMD:C_0402_1005Metric -> Capacitor_SMD:C_0201_0603Metric; JLCPCB_CORRECTION 0;0;0 -> (none); LCSC C1518208 -> C76935; info 50V, X5R (potenciálně C52923 což je 25V, X5R ) -> 10V, X5R
- J2: footprint Connector_JST:JST_PH_S2B-PH-SM4-TB_1x02-1MP_P2.00mm_Horizontal -> Connector_PinHeader_2.00mm:PinHeader_1x02_P2.00mm_Vertical
- Q2, Q7, U2: Basic/Extended (none) -> E
- R10, R15: footprint Resistor_SMD:R_0402_1005Metric -> Resistor_SMD:R_0201_0603Metric; Basic/Extended B -> E; LCSC C25764 -> C171922
- R13, R19: footprint Resistor_SMD:R_0402_1005Metric -> Resistor_SMD:R_0201_0603Metric; Basic/Extended B -> E; LCSC C26083 -> C295786
- R16, R17, R25: footprint Resistor_SMD:R_0402_1005Metric -> Resistor_SMD:R_0201_0603Metric; Basic/Extended B -> E; JLCPCB_CORRECTION 0;0;0 -> (none); LCSC C25744 -> C106225
Other:
- moved on the sheet: C9, Q?, R10, R16, R17, R18, R19, R25, SW4

Commit message: PCB
Parts:
- added C35: 1u, Capacitor_SMD:C_0402_1005Metric, symbol Device:C
- C7: footprint Capacitor_SMD:C_0201_0603Metric -> Capacitor_SMD:C_0402_1005Metric; Basic/Extended E -> B; LCSC C5142565 -> C307331; info 10V, X5R -> 50V, X7R
- C8, C9: footprint Capacitor_SMD:C_0201_0603Metric -> Capacitor_SMD:C_0402_1005Metric; Basic/Extended E -> B; LCSC C76935 -> C52923; info 10V, X5R -> 25V, X5R
- R10, R15: footprint Resistor_SMD:R_0201_0603Metric -> Resistor_SMD:R_0402_1005Metric; Basic/Extended E -> B; LCSC C171922 -> C25764
- R13, R19: footprint Resistor_SMD:R_0201_0603Metric -> Resistor_SMD:R_0402_1005Metric; Basic/Extended E -> B; LCSC C295786 -> C26083
- R16, R17, R25: footprint Resistor_SMD:R_0201_0603Metric -> Resistor_SMD:R_0402_1005Metric; Basic/Extended E -> B; LCSC C106225 -> C25744
Connections:
- net VCC: now also C35.1
- net at Q?.2 (G), Q?.2 (G), R25.2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: now also C35.2
Other:
- moved on the sheet: SW4
