File: hw/Watch/MainBoard/Charger.kicad_sch (KiCad schematic)
At the start: 13 parts, among them U5 10u, U6 10u, U7 10u, U8 BQ25895RTW

Commit message: WIP
Parts:
- L1: footprint Inductor_SMD:L_Abracon_ASPI-0630LR -> Inductor_SMD:L_1008_2520Metric; LCSC C5307644 -> C1017131
Changed lines of the file:
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@@
       (effects (font (size 1.27 1.27)))
     )
-    (property "Footprint" "Inductor_SMD:L_Abracon_ASPI-0630LR" (at 166.37 68.58 0)
+    (property "Footprint" "Inductor_SMD:L_1008_2520Metric" (at 166.37 68.58 0)
       (effects (font (size 1.27 1.27)) hide)
     )
@@
       (effects (font (size 1.27 1.27)) hide)
     )
-    (property "LCSC" "C5307644" (at 166.37 68.58 90)
+    (property "LCSC" "C1017131" (at 166.37 68.58 90)
       (effects (font (size 1.27 1.27)) hide)
     )

Commit message: wip
Parts:
- added C32, C33: 10u, Capacitor_SMD:C_0402_1005Metric, symbol Device:C
- C24: footprint Capacitor_SMD:C_0402_1005Metric -> Capacitor_SMD:C_0201_0603Metric; JLCPCB_CORRECTION 0;0;0 -> (none); LCSC C1518208 -> C76935; info 50V, X5R (potenciálně C52923 což je 25V, X5R ) -> 10V, X5R
- C25: footprint Capacitor_SMD:C_0603_1608Metric -> Capacitor_SMD:C_0201_0603Metric; Basic/Extended B -> E; LCSC C1622 -> C5142564; info 50V, X7R -> 25V, X5R
- C26: footprint Capacitor_SMD:C_0603_1608Metric -> Capacitor_SMD:C_0402_1005Metric; LCSC C19666 -> C23733
- C29: renamed from U5; footprint Capacitor_SMD:C_0603_1608Metric -> Capacitor_SMD:C_0402_1005Metric; Basic/Extended B -> E; LCSC C96446 -> C315248; info 25V, X5R -> 10V, X5R
- C30: renamed from U6; footprint Capacitor_SMD:C_0603_1608Metric -> Capacitor_SMD:C_0402_1005Metric; Basic/Extended B -> E; LCSC C96446 -> C315248; info 25V, X5R -> 10V, X5R
- C31: renamed from U7; footprint Capacitor_SMD:C_0603_1608Metric -> Capacitor_SMD:C_0402_1005Metric; Basic/Extended B -> E; LCSC C96446 -> C315248; info 25V, X5R -> 10V, X5R
- R22, R26: footprint Resistor_SMD:R_0402_1005Metric -> Resistor_SMD:R_0201_0603Metric; Basic/Extended B -> E; JLCPCB_CORRECTION 0;0;0 -> (none); LCSC C25744 -> C106225
Connections:
- net 5V: now also C32.1, C33.1
- net GND: now also C32.2, C33.2

Commit message: PCB
Parts:
- C24: footprint Capacitor_SMD:C_0201_0603Metric -> Capacitor_SMD:C_0402_1005Metric; Basic/Extended E -> B; LCSC C76935 -> C52923; info 10V, X5R -> 25V, X5R
- R21: value 4.7k -> 2k; LCSC C25900 -> C4109
- R22, R26: footprint Resistor_SMD:R_0201_0603Metric -> Resistor_SMD:R_0402_1005Metric; Basic/Extended E -> B; LCSC C106225 -> C25744
Connections:
- net STAT: now also D14.2 (A); no longer R21.1
- net at R21.2: now also C29.1, C30.1, L1.2, U8.15 (SYS), U8.16 (SYS); no longer D14.2 (A)
- new net: D14.1 (K), R21.1
Other:
- moved on the sheet: D14, R21
Changed lines of the file:
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@@
     (effects (font (size 1.27 1.27)) (justify right))
   )
-  (symbol (lib_id "Device:R") (at 172.72 92.71 180) (unit 1)
-    (in_bom yes) (on_board yes) (dnp no)
-    (property "Reference" "R21" (at 168.91 91.44 0)
-      (effects (font (size 1.27 1.27)))
-    )
-    (property "Value" "4.7k" (at 168.91 93.98 0)
-      (effects (font (size 1.27 1.27)))
-    )
-    (property "Footprint" "Resistor_SMD:R_0402_1005Metric" (at 174.498 92.71 90)
-      (effects (font (size 1.27 1.27)) hide)
-    )
-    (property "Datasheet" "~" (at 172.72 92.71 0)
-      (effects (font (size 1.27 1.27)) hide)
-    )
-    (property "LCSC" "C25900" (at 172.72 92.71 0)
-      (effects (font (size 1.27 1.27)) hide)
-    )
-    (property "Basic/Extended" "B" (at 172.72 92.71 0)
+  (symbol (lib_id "Device:R") (at 172.72 85.09 180) (unit 1)
+    (in_bom yes) (on_board yes) (dnp no)
+    (property "Reference" "R21" (at 168.91 83.82 0)
+      (effects (font (size 1.27 1.27)))
+    )
+    (property "Value" "2k" (at 168.91 86.36 0)
+      (effects (font (size 1.27 1.27)))
+    )
+    (property "Footprint" "Resistor_SMD:R_0402_1005Metric" (at 174.498 85.09 90)
+      (effects (font (size 1.27 1.27)) hide)
+    )
+    (property "Datasheet" "~" (at 172.72 85.09 0)
+      (effects (font (size 1.27 1.27)) hide)
+    )
+    (property "LCSC" "C4109" (at 172.72 85.09 0)
+      (effects (font (size 1.27 1.27)) hide)
+    )
+    (property "Basic/Extended" "B" (at 172.72 85.09 0)
       (effects (font (size 1.27 1.27)) hide)
     )
@@
       (effects (font (size 1.27 1.27)) (justify left))
     )
-    (property "Footprint" "Capacitor_SMD:C_0201_0603Metric" (at 102.5652 73.66 0)
+    (property "Footprint" "Capacitor_SMD:C_0402_1005Metric" (at 102.5652 73.66 0)
       (effects (font (size 1.27 1.27)) hide)
     )
@@
       (effects (font (size 1.27 1.27)) hide)
     )
-    (property "LCSC" "C76935" (at 101.6 69.85 0)
-      (effects (font (size 1.27 1.27)) hide)
-    )
-    (property "info" "10V, X5R" (at 101.6 69.85 0)
-      (effects (font (size 1.27 1.27)) hide)
-    )
-    (property "Basic/Extended" "E" (at 101.6 69.85 0)
+    (property "LCSC" "C52923" (at 101.6 69.85 0)
+      (effects (font (size 1.27 1.27)) hide)
+    )
+    (property "info" "25V, X5R" (at 101.6 69.85 0)
+      (effects (font (size 1.27 1.27)) hide)
+    )
+    (property "Basic/Extended" "B" (at 101.6 69.85 0)
       (effects (font (size 1.27 1.27)) hide)
     )
@@
     )
   )
-  (symbol (lib_id "Device:LED") (at 172.72 85.09 270) (unit 1)
-    (in_bom yes) (on_board yes) (dnp no)
-    (property "Reference" "D14" (at 167.64 83.82 90)
-      (effects (font (size 1.27 1.27)))
-    )
-    (property "Value" "red" (at 167.64 86.36 90)
-      (effects (font (size 1.27 1.27)))
-    )
-    (property "Footprint" "LED_SMD:LED_0603_1608Metric" (at 172.72 85.09 0)
-      (effects (font (size 1.27 1.27)) hide)
-    )
-    (property "Datasheet" "~" (at 172.72 85.09 0)
-      (effects (font (size 1.27 1.27)) hide)
-    )
-    (property "LCSC" "C2286" (at 172.72 85.09 90)
-      (effects (font (size 1.27 1.27)) hide)
-    )
-    (property "Basic/Extended" "B" (at 172.72 85.09 90)
+  (symbol (lib_id "Device:LED") (at 172.72 92.71 270) (unit 1)
+    (in_bom yes) (on_board yes) (dnp no)
+    (property "Reference" "D14" (at 167.64 91.44 90)
+      (effects (font (size 1.27 1.27)))
+    )
+    (property "Value" "red" (at 167.64 93.98 90)
+      (effects (font (size 1.27 1.27)))
+    )
+    (property "Footprint" "LED_SMD:LED_0603_1608Metric" (at 172.72 92.71 0)
+      (effects (font (size 1.27 1.27)) hide)
+    )
+    (property "Datasheet" "~" (at 172.72 92.71 0)
+      (effects (font (size 1.27 1.27)) hide)
+    )
+    (property "LCSC" "C2286" (at 172.72 92.71 90)
+      (effects (font (size 1.27 1.27)) hide)
+    )
+    (property "Basic/Extended" "B" (at 172.72 92.71 90)
       (effects (font (size 1.27 1.27)) hide)
     )
@@
       (effects (font (size 1.27 1.27)) (justify left))
     )
-    (property "Footprint" "Resistor_SMD:R_0201_0603Metric" (at 150.622 105.41 90)
+    (property "Footprint" "Resistor_SMD:R_0402_1005Metric" (at 150.622 105.41 90)
       (effects (font (size 1.27 1.27)) hide)
     )
@@
       (effects (font (size 1.27 1.27)) hide)
     )
-    (property "LCSC" "C106225" (at 152.4 105.41 0)
-      (effects (font (size 1.27 1.27)) hide)
-    )
-    (property "Basic/Extended" "E" (at 152.4 105.41 0)
+    (property "LCSC" "C25744" (at 152.4 105.41 0)
+      (effects (font (size 1.27 1.27)) hide)
+    )
+    (property "Basic/Extended" "B" (at 152.4 105.41 0)
       (effects (font (size 1.27 1.27)) hide)
     )
@@
       (effects (font (size 1.27 1.27)) (justify left))
     )
-    (property "Footprint" "Resistor_SMD:R_0201_0603Metric" (at 158.75 100.838 90)
+    (property "Footprint" "Resistor_SMD:R_0402_1005Metric" (at 158.75 100.838 90)
       (effects (font (size 1.27 1.27)) hide)
     )
@@
       (effects (font (size 1.27 1.27)) hide)
     )
-    (property "LCSC" "C106225" (at 158.75 99.06 0)
-      (effects (font (size 1.27 1.27)) hide)
-    )
-    (property "Basic/Extended" "E" (at 158.75 99.06 0)
-      (effects (font (size 1.27 1.27)) hide)
-    )
+    (property "LCSC" "C25744" (at 158.75 99.06 0)
+      (effects (font (size 1.27 1.27)) hide)
+    )
+    (property "Basic/Extended" "B" (at 158.75 99.06 0)
+      (effects (font (size 1.27 1.27)) hide)
+    )

Commit message: PCB v0.0.0
Parts:
- renumbered L1 to L3
Changed lines of the file:
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@@
   (symbol (lib_id "Device:L") (at 166.37 68.58 90) (unit 1)
     (in_bom yes) (on_board yes) (dnp no)
-    (property "Reference" "L1" (at 166.37 66.04 90)
+    (property "Reference" "L3" (at 166.37 66.04 90)
       (effects (font (size 1.27 1.27)))
     )
@@
       (project "Watch"
         (path "/1db6f6a7-b341-422f-8dcc-b4fd8e3ba0c0/7a0b441f-fb08-4406-ad74-ba91736d76e3/e51762e8-40da-4e3a-afe4-857a6428bc26/6f1fd0d6-76d4-4e62-b397-b40d00c396e2"
-          (reference "L1") (unit 1)
+          (reference "L3") (unit 1)
         )
       )
