File: hw/Watch/MainBoard/USB.kicad_sch (KiCad schematic)
At the start: 5 parts, among them J2 USB_C_Receptacle_USB2.0, U9 TPD4E02B04DQA

Commit message: wip
Parts:
- removed D15: PTVSHC3N24, RKL-StandardPackages:DFN3-2x2, symbol RKL-Uncategorized:PTVSHC3N24
Changed lines of the file:
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@@
   (junction (at 139.7 63.5) (diameter 0) (color 0 0 0 0)
-  )
-  (junction (at 177.8 63.5) (diameter 0) (color 0 0 0 0)
   )
   (junction (at 142.24 81.28) (diameter 0) (color 0 0 0 0)
@@
     (stroke (width 0) (type default))
   )
-  (wire (pts (xy 177.8 81.28) (xy 177.8 78.74))
-    (stroke (width 0) (type default))
-  )
   (wire (pts (xy 129.54 83.82) (xy 129.54 81.28))
     (stroke (width 0) (type default))
@@
     (stroke (width 0) (type default))
   )
-  (wire (pts (xy 177.8 63.5) (xy 190.5 63.5))
-    (stroke (width 0) (type default))
-  )
   (wire (pts (xy 142.24 81.28) (xy 144.78 81.28))
     (stroke (width 0) (type default))
@@
   )
   (wire (pts (xy 127 68.58) (xy 132.08 68.58))
-    (stroke (width 0) (type default))
-  )
-  (wire (pts (xy 177.8 63.5) (xy 177.8 71.12))
     (stroke (width 0) (type default))
   )
@@
     (effects (font (size 1.27 1.27)) (justify left))
   )
-  (hierarchical_label "GND" (shape bidirectional) (at 177.8 81.28 270) (fields_autoplaced)
-    (effects (font (size 1.27 1.27)) (justify right))
-  )
   (hierarchical_label "GND" (shape bidirectional) (at 161.29 81.28 270) (fields_autoplaced)
     (effects (font (size 1.27 1.27)) (justify right))
   )
-  (hierarchical_label "VBUS" (shape input) (at 190.5 63.5 0) (fields_autoplaced)
+  (hierarchical_label "VBUS" (shape input) (at 177.8 63.5 0) (fields_autoplaced)
     (effects (font (size 1.27 1.27)) (justify left))
   )
@@
         )
       )
-    )
-  )
-  (symbol (lib_id "RKL-Uncategorized:PTVSHC3N24") (at 177.8 74.93 270) (mirror x) (unit 1)
-    (in_bom yes) (on_board yes) (dnp no)
-    (property "Reference" "D15" (at 180.34 73.66 90)
-      (effects (font (size 1.27 1.27)) (justify left))
-    )
-    (property "Value" "PTVSHC3N24" (at 180.34 76.2 90)
-      (effects (font (size 1.27 1.27)) (justify left))
-    )
-    (property "Footprint" "RKL-StandardPackages:DFN3-2x2" (at 194.31 74.93 0)
-      (effects (font (size 1.27 1.27)) hide)
-    )
-    (property "Datasheet" "https://datasheet.lcsc.com/lcsc/2012241239_Shanghai-Prisemi-Elec-PTVSHC3N24VUH_C1021680.pdf" (at 190.5 74.93 0)
-      (effects (font (size 1.27 1.27)) hide)
-    )
-    (property "LCSC" "C312228" (at 186.69 74.93 0)
-      (effects (font (size 1.27 1.27)) hide)
-    )
-    (property "Basic/Extended" "E" (at 177.8 74.93 0)
-      (effects (font (size 1.27 1.27)) hide)
-    )
-    (pin "1")
-    (pin "2")
-    (pin "3")
-    (instances
-      (project "Watch"
-        (path "/1db6f6a7-b341-422f-8dcc-b4fd8e3ba0c0/7a0b441f-fb08-4406-ad74-ba91736d76e3/8404aa54-70b5-4b05-b451-94d119f275f2"
-          (reference "D15") (unit 1)
-        )
-      )
-      (project "ZakladniElektronika"
-        (path "/99cd3e15-4eb6-4cbb-8726-789aedd3df15/c3b70d9b-0dcb-4344-9507-13ff5b4c000e/2f609c37-b91c-437d-a066-c26014011f90"
-          (reference "D123") (unit 1)
-        )
-      )
-      (project "RB3203"
-        (path "/dc7f8a41-3453-4df6-94dc-e94521e89591/9c917b4f-c6c7-4191-9aaa-f982c264da50/42c6643c-04e2-43ad-8f0e-80e5d3fe214b"
-          (reference "D?") (unit 1)
-        )
-      )

Commit message: WIP
Parts:
- removed J2: USB_C_Receptacle_USB2.0, RKL-Connectors:USB31-TYPEC-33141-2FS, symbol Connector:USB_C_Receptacle
- added J7: USB_C_Receptacle_USB2.0, RKL-Connectors:USB-C_vertical, symbol Connector:USB_C_Receptacle_USB2.0
Connections:
- net D+: now also J7.A6 (D+), J7.B6 (D+)
- net D-: now also J7.A7 (D-), J7.B7 (D-)
- net GND: now also J7.A1 (GND), J7.A12 (GND), J7.B1 (GND), J7.B12 (GND), J7.S1 (SHIELD)
- net USB_CC1: now also J7.A5 (CC1)
- net USB_CC2: now also J7.B5 (CC2)
- net VBUS: now also J7.A4 (VBUS), J7.A9 (VBUS), J7.B4 (VBUS), J7.B9 (VBUS)
- no-connect marks 10 -> 2
Changed lines of the file:
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@@
   (junction (at 132.08 68.58) (diameter 0) (color 0 0 0 0)
   )
-  (no_connect (at 127 99.06))
-  (no_connect (at 127 106.68))
-  (no_connect (at 127 111.76))
-  (no_connect (at 127 104.14))
-  (no_connect (at 127 96.52))
-  (no_connect (at 127 88.9))
-  (no_connect (at 127 121.92))
-  (no_connect (at 127 119.38))
-  (no_connect (at 127 114.3))
   (no_connect (at 127 91.44))
+  (no_connect (at 127 93.98))
   (wire (pts (xy 139.7 78.74) (xy 139.7 86.36))
     (stroke (width 0) (type default))
@@
     (effects (font (size 1.27 1.27)) (justify left bottom))
   )
-  (hierarchical_label "GND" (shape bidirectional) (at 104.14 129.54 270) (fields_autoplaced)
+  (hierarchical_label "GND" (shape bidirectional) (at 104.14 101.6 270) (fields_autoplaced)
     (effects (font (size 1.27 1.27)) (justify right))
   )
@@
     (effects (font (size 1.27 1.27)) (justify left))
   )
-  (hierarchical_label "GND" (shape bidirectional) (at 111.76 129.54 270) (fields_autoplaced)
+  (hierarchical_label "GND" (shape bidirectional) (at 111.76 101.6 270) (fields_autoplaced)
     (effects (font (size 1.27 1.27)) (justify right))
   )
@@
     )
   )
-  (symbol (lib_id "Device:R") (at 165.1 77.47 0) (unit 1)
+  (symbol (lib_id "Connector:USB_C_Receptacle_USB2.0") (at 111.76 78.74 0) (unit 1)
     (in_bom yes) (on_board yes) (dnp no) (fields_autoplaced)
-    (property "Reference" "R24" (at 167.64 76.1999 0)
-      (effects (font (size 1.27 1.27)) (justify left))
-    )
-    (property "Value" "5.1k" (at 167.64 78.7399 0)
-      (effects (font (size 1.27 1.27)) (justify left))
-    )
-    (property "Footprint" "Resistor_SMD:R_0402_1005Metric" (at 163.322 77.47 90)
-      (effects (font (size 1.27 1.27)) hide)
-    )
-    (property "Datasheet" "~" (at 165.1 77.47 0)
-      (effects (font (size 1.27 1.27)) hide)
-    )
-    (property "LCSC" "C25905" (at 165.1 77.47 0)
-      (effects (font (size 1.27 1.27)) hide)
-    )
-    (property "Basic/Extended" "B" (at 165.1 77.47 0)
-      (effects (font (size 1.27 1.27)) hide)
-    )
-    (pin "1")
-    (pin "2")
-    (instances
-      (project "Watch"
-        (path "/1db6f6a7-b341-422f-8dcc-b4fd8e3ba0c0/7a0b441f-fb08-4406-ad74-ba91736d76e3/8404aa54-70b5-4b05-b451-94d119f275f2"
-          (reference "R24") (unit 1)
-        )
-      )
-      (project "ZakladniElektronika"
-        (path "/99cd3e15-4eb6-4cbb-8726-789aedd3df15/c3b70d9b-0dcb-4344-9507-13ff5b4c000e/2f609c37-b91c-437d-a066-c26014011f90"
-          (reference "R4") (unit 1)
-        )
-      )
-      (project "RB3203"
-        (path "/dc7f8a41-3453-4df6-94dc-e94521e89591/9c917b4f-c6c7-4191-9aaa-f982c264da50/42c6643c-04e2-43ad-8f0e-80e5d3fe214b"
-          (reference "R?") (unit 1)
-        )
-      )
-    )
-  )
-  (symbol (lib_id "Connector:USB_C_Receptacle") (at 111.76 88.9 0) (unit 1)
-    (in_bom yes) (on_board yes) (dnp no)
-    (property "Reference" "J2" (at 111.76 57.15 0)
+    (property "Reference" "J7" (at 111.76 55.88 0)
       (effects (font (size 1.27 1.27)))
     )
-    (property "Value" "USB_C_Receptacle_USB2.0" (at 114.4778 59.0296 0)
+    (property "Value" "USB_C_Receptacle_USB2.0" (at 111.76 58.42 0)
       (effects (font (size 1.27 1.27)))
     )
-    (property "Footprint" "RKL-Connectors:USB31-TYPEC-33141-2FS" (at 115.57 88.9 0)
-      (effects (font (size 1.27 1.27)) hide)
-    )
-    (property "Datasheet" "https://www.usb.org/sites/default/files/documents/usb_type-c.zip" (at 115.57 88.9 0)
-      (effects (font (size 1.27 1.27)) hide)
-    )
-    (property "LCSC" "C480368" (at 111.76 59.69 0)
-      (effects (font (size 1.27 1.27)) hide)
-    )
-    (property "JLCPCB_CORRECTION" "0;-3.5;0" (at 111.76 54.61 0)
-      (effects (font (size 1.27 1.27)) hide)
-    )
-    (property "Basic/Extended" "E" (at 111.76 57.15 0)
+    (property "Footprint" "RKL-Connectors:USB-C_vertical" (at 115.57 78.74 0)
+      (effects (font (size 1.27 1.27)) hide)
+    )
+    (property "Datasheet" "https://www.usb.org/sites/default/files/documents/usb_type-c.zip" (at 115.57 78.74 0)
       (effects (font (size 1.27 1.27)) hide)
     )
     (pin "A1")
-    (pin "A10")
-    (pin "A11")
     (pin "A12")
-    (pin "A2")
-    (pin "A3")
     (pin "A4")
     (pin "A5")
@@
     (pin "A9")
     (pin "B1")
-    (pin "B10")
-    (pin "B11")
     (pin "B12")
-    (pin "B2")
-    (pin "B3")
     (pin "B4")
     (pin "B5")
@@
       (project "Watch"
         (path "/1db6f6a7-b341-422f-8dcc-b4fd8e3ba0c0/7a0b441f-fb08-4406-ad74-ba91736d76e3/8404aa54-70b5-4b05-b451-94d119f275f2"
-          (reference "J2") (unit 1)
+          (reference "J7") (unit 1)
+        )
+      )
+    )
+  )
+  (symbol (lib_id "Device:R") (at 165.1 77.47 0) (unit 1)
+    (in_bom yes) (on_board yes) (dnp no) (fields_autoplaced)
+    (property "Reference" "R24" (at 167.64 76.1999 0)
+      (effects (font (size 1.27 1.27)) (justify left))
+    )
+    (property "Value" "5.1k" (at 167.64 78.7399 0)
+      (effects (font (size 1.27 1.27)) (justify left))
+    )
+    (property "Footprint" "Resistor_SMD:R_0402_1005Metric" (at 163.322 77.47 90)
+      (effects (font (size 1.27 1.27)) hide)
+    )
+    (property "Datasheet" "~" (at 165.1 77.47 0)
+      (effects (font (size 1.27 1.27)) hide)
+    )
+    (property "LCSC" "C25905" (at 165.1 77.47 0)
+      (effects (font (size 1.27 1.27)) hide)
+    )
+    (property "Basic/Extended" "B" (at 165.1 77.47 0)
+      (effects (font (size 1.27 1.27)) hide)
+    )
+    (pin "1")
+    (pin "2")
+    (instances
+      (project "Watch"
+        (path "/1db6f6a7-b341-422f-8dcc-b4fd8e3ba0c0/7a0b441f-fb08-4406-ad74-ba91736d76e3/8404aa54-70b5-4b05-b451-94d119f275f2"
+          (reference "R24") (unit 1)
         )
       )
       (project "ZakladniElektronika"
         (path "/99cd3e15-4eb6-4cbb-8726-789aedd3df15/c3b70d9b-0dcb-4344-9507-13ff5b4c000e/2f609c37-b91c-437d-a066-c26014011f90"
-          (reference "J2") (unit 1)
+          (reference "R4") (unit 1)
         )
       )
       (project "RB3203"
         (path "/dc7f8a41-3453-4df6-94dc-e94521e89591/9c917b4f-c6c7-4191-9aaa-f982c264da50/42c6643c-04e2-43ad-8f0e-80e5d3fe214b"
-          (reference "J?") (unit 1)
-        )
-      )
+          (reference "R?") (unit 1)
+        )
+      )

Commit message: wip
Parts:
- added C26: 4.7u, Capacitor_SMD:C_0402_1005Metric, symbol Device:C
- J7: Basic/Extended (none) -> E; LCSC (none) -> C2686963
- R12, R24: footprint Resistor_SMD:R_0402_1005Metric -> Resistor_SMD:R_0201_0603Metric; Basic/Extended B -> E; LCSC C25905 -> C163490
Connections:
- net GND: now also C26.2
- net USB_CC1: no longer U9.1 (IO1)
- net USB_CC2: no longer U9.2 (IO2)
- net VBUS: now also U9.1 (IO1), U9.2 (IO2), C26.1
Changed lines of the file:
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@@
 (kicad_sch (version 20230121) (generator eeschema)
   (paper "A4")
+  (junction (at 132.08 83.82) (diameter 0) (color 0 0 0 0)
+  )
   (junction (at 139.7 78.74) (diameter 0) (color 0 0 0 0)
   )
@@
   (junction (at 129.54 81.28) (diameter 0) (color 0 0 0 0)
   )
-  (junction (at 134.62 71.12) (diameter 0) (color 0 0 0 0)
+  (junction (at 177.8 63.5) (diameter 0) (color 0 0 0 0)
   )
   (junction (at 139.7 63.5) (diameter 0) (color 0 0 0 0)
   )
+  (junction (at 132.08 63.5) (diameter 0) (color 0 0 0 0)
+  )
   (junction (at 142.24 81.28) (diameter 0) (color 0 0 0 0)
-  )
-  (junction (at 132.08 68.58) (diameter 0) (color 0 0 0 0)
   )
   (no_connect (at 127 91.44))
   (no_connect (at 127 93.98))
+  (wire (pts (xy 177.8 63.5) (xy 190.5 63.5))
+    (stroke (width 0) (type default))
+  )
+  (wire (pts (xy 134.62 86.36) (xy 134.62 83.82))
+    (stroke (width 0) (type default))
+  )
   (wire (pts (xy 139.7 78.74) (xy 139.7 86.36))
     (stroke (width 0) (type default))
@@
     (stroke (width 0) (type default))
   )
+  (wire (pts (xy 134.62 83.82) (xy 132.08 83.82))
+    (stroke (width 0) (type default))
+  )
   (wire (pts (xy 142.24 81.28) (xy 142.24 86.36))
     (stroke (width 0) (type default))
   )
+  (wire (pts (xy 132.08 83.82) (xy 132.08 86.36))
+    (stroke (width 0) (type default))
+  )
   (wire (pts (xy 165.1 68.58) (xy 165.1 73.66))
     (stroke (width 0) (type default))
@@
     (stroke (width 0) (type default))
   )
+  (wire (pts (xy 132.08 63.5) (xy 139.7 63.5))
+    (stroke (width 0) (type default))
+  )
+  (wire (pts (xy 132.08 63.5) (xy 132.08 83.82))
+    (stroke (width 0) (type default))
+  )
   (wire (pts (xy 129.54 78.74) (xy 129.54 76.2))
     (stroke (width 0) (type default))
   )
-  (wire (pts (xy 134.62 71.12) (xy 134.62 86.36))
-    (stroke (width 0) (type default))
-  )
   (wire (pts (xy 129.54 81.28) (xy 142.24 81.28))
     (stroke (width 0) (type default))
   )
-  (wire (pts (xy 127 71.12) (xy 134.62 71.12))
+  (wire (pts (xy 127 71.12) (xy 161.29 71.12))
     (stroke (width 0) (type default))
   )
@@
     (stroke (width 0) (type default))
   )
-  (wire (pts (xy 132.08 68.58) (xy 132.08 86.36))
-    (stroke (width 0) (type default))
-  )
-  (wire (pts (xy 132.08 68.58) (xy 165.1 68.58))
-    (stroke (width 0) (type default))
-  )
-  (wire (pts (xy 127 68.58) (xy 132.08 68.58))
-    (stroke (width 0) (type default))
-  )
-  (wire (pts (xy 127 63.5) (xy 139.7 63.5))
+  (wire (pts (xy 177.8 63.5) (xy 177.8 73.66))
+    (stroke (width 0) (type default))
+  )
+  (wire (pts (xy 127 68.58) (xy 165.1 68.58))
+    (stroke (width 0) (type default))
+  )
+  (wire (pts (xy 127 63.5) (xy 132.08 63.5))
     (stroke (width 0) (type default))
   )
   (wire (pts (xy 139.7 78.74) (xy 144.78 78.74))
-    (stroke (width 0) (type default))
-  )
-  (wire (pts (xy 134.62 71.12) (xy 161.29 71.12))
     (stroke (width 0) (type default))
   )
@@
     (effects (font (size 1.27 1.27)) (justify left bottom))
   )
-  (label "V_USB" (at 144.78 63.5 0) (fields_autoplaced)
+  (label "VBUS" (at 144.78 63.5 0) (fields_autoplaced)
     (effects (font (size 1.27 1.27)) (justify left bottom))
   )
@@
     (effects (font (size 1.27 1.27)) (justify right))
   )
-  (hierarchical_label "VBUS" (shape input) (at 177.8 63.5 0) (fields_autoplaced)
+  (hierarchical_label "GND" (shape bidirectional) (at 177.8 81.28 270) (fields_autoplaced)
+    (effects (font (size 1.27 1.27)) (justify right))
+  )
+  (hierarchical_label "VBUS" (shape input) (at 190.5 63.5 0) (fields_autoplaced)
     (effects (font (size 1.27 1.27)) (justify left))
   )
@@
     )
     (property "Datasheet" "https://www.usb.org/sites/default/files/documents/usb_type-c.zip" (at 115.57 78.74 0)
+      (effects (font (size 1.27 1.27)) hide)
+    )
+    (property "Basic/Extended" "E" (at 111.76 78.74 0)
+      (effects (font (size 1.27 1.27)) hide)
+    )
+    (property "LCSC" "C2686963" (at 111.76 78.74 0)
       (effects (font (size 1.27 1.27)) hide)
     )
@@
       (effects (font (size 1.27 1.27)) (justify left))
     )
-    (property "Footprint" "Resistor_SMD:R_0402_1005Metric" (at 163.322 77.47 90)
+    (property "Footprint" "Resistor_SMD:R_0201_0603Metric" (at 163.322 77.47 90)
       (effects (font (size 1.27 1.27)) hide)
     )
@@
       (effects (font (size 1.27 1.27)) hide)
     )
-    (property "LCSC" "C25905" (at 165.1 77.47 0)
-      (effects (font (size 1.27 1.27)) hide)
-    )
-    (property "Basic/Extended" "B" (at 165.1 77.47 0)
+    (property "LCSC" "C163490" (at 165.1 77.47 0)
+      (effects (font (size 1.27 1.27)) hide)
+    )
+    (property "Basic/Extended" "E" (at 165.1 77.47 0)
       (effects (font (size 1.27 1.27)) hide)
     )
@@
     )
   )
+  (symbol (lib_id "Device:C") (at 177.8 77.47 0) (unit 1)
+    (in_bom yes) (on_board yes) (dnp no)
+    (property "Reference" "C26" (at 180.721 76.3016 0)
+      (effects (font (size 1.27 1.27)) (justify left))
+    )
+    (property "Value" "4.7u" (at 180.721 78.613 0)
+      (effects (font (size 1.27 1.27)) (justify left))
+    )
+    (property "Footprint" "Capacitor_SMD:C_0402_1005Metric" (at 178.7652 81.28 0)
+      (effects (font (size 1.27 1.27)) hide)
+    )
+    (property "Datasheet" "~" (at 177.8 77.47 0)
+      (effects (font (size 1.27 1.27)) hide)
+    )
+    (property "LCSC" "C23733" (at 177.8 77.47 0)
+      (effects (font (size 1.27 1.27)) hide)
+    )
+    (property "Basic/Extended" "B" (at 177.8 77.47 0)
+      (effects (font (size 1.27 1.27)) hide)
+    )
+    (property "info" "16V, X5R" (at 177.8 77.47 0)
+      (effects (font (size 1.27 1.27)) hide)
+    )
+    (pin "1")
+    (pin "2")
+    (instances
+      (project "Watch"
+        (path "/1db6f6a7-b341-422f-8dcc-b4fd8e3ba0c0/7a0b441f-fb08-4406-ad74-ba91736d76e3/e51762e8-40da-4e3a-afe4-857a6428bc26/6f1fd0d6-76d4-4e62-b397-b40d00c396e2"
+          (reference "C26") (unit 1)
+        )
+        (path "/1db6f6a7-b341-422f-8dcc-b4fd8e3ba0c0/7a0b441f-fb08-4406-ad74-ba91736d76e3/8404aa54-70b5-4b05-b451-94d119f275f2"
+          (reference "C34") (unit 1)
+        )
+      )
+      (project "ZakladniElektronika"
+        (path "/99cd3e15-4eb6-4cbb-8726-789aedd3df15/c3b70d9b-0dcb-4344-9507-13ff5b4c000e/aae02708-da26-44dd-a602-660fbe003309/3940fef8-969a-4db4-8b0b-434b96d98566"
+          (reference "C150") (unit 1)
+        )
+        (path "/99cd3e15-4eb6-4cbb-8726-789aedd3df15/c3b70d9b-0dcb-4344-9507-13ff5b4c000e/aae02708-da26-44dd-a602-660fbe003309/4ff5c299-eafc-48ae-8fce-c1c1f5f569e7"
+          (reference "C164") (unit 1)
+        )
+      )
+      (project "RB3203"
+        (path "/dc7f8a41-3453-4df6-94dc-e94521e89591/9c917b4f-c6c7-4191-9aaa-f982c264da50/8773969d-b2cc-42c4-9a6d-35c6f165cf16/da5be375-027b-4f55-96f0-042c23671c4c"
+          (reference "U?") (unit 1)
+        )
+      )
+    )
+  )
   (symbol (lib_id "Device:R") (at 161.29 77.47 0) (unit 1)
     (in_bom yes) (on_board yes) (dnp no)
@@
       (effects (font (size 1.27 1.27)) (justify left))
     )
-    (property "Footprint" "Resistor_SMD:R_0402_1005Metric" (at 159.512 77.47 90)
+    (property "Footprint" "Resistor_SMD:R_0201_0603Metric" (at 159.512 77.47 90)
       (effects (font (size 1.27 1.27)) hide)
     )
@@
       (effects (font (size 1.27 1.27)) hide)
     )
-    (property "LCSC" "C25905" (at 161.29 77.47 0)
-      (effects (font (size 1.27 1.27)) hide)
-    )
-    (property "Basic/Extended" "B" (at 161.29 77.47 0)
-      (effects (font (size 1.27 1.27)) hide)
-    )
+    (property "LCSC" "C163490" (at 161.29 77.47 0)
+      (effects (font (size 1.27 1.27)) hide)
+    )
+    (property "Basic/Extended" "E" (at 161.29 77.47 0)
+      (effects (font (size 1.27 1.27)) hide)
+    )

Commit message: PCB
Parts:
- R12, R24: footprint Resistor_SMD:R_0201_0603Metric -> Resistor_SMD:R_0402_1005Metric; Basic/Extended E -> B; LCSC C163490 -> C25905
Changed lines of the file:
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@@
       (effects (font (size 1.27 1.27)) (justify left))
     )
-    (property "Footprint" "Resistor_SMD:R_0201_0603Metric" (at 163.322 77.47 90)
+    (property "Footprint" "Resistor_SMD:R_0402_1005Metric" (at 163.322 77.47 90)
       (effects (font (size 1.27 1.27)) hide)
     )
@@
       (effects (font (size 1.27 1.27)) hide)
     )
-    (property "LCSC" "C163490" (at 165.1 77.47 0)
+    (property "LCSC" "C25905" (at 165.1 77.47 0)
       (effects (font (size 1.27 1.27)) hide)
     )
-    (property "Basic/Extended" "E" (at 165.1 77.47 0)
+    (property "Basic/Extended" "B" (at 165.1 77.47 0)
       (effects (font (size 1.27 1.27)) hide)
     )
@@
       (effects (font (size 1.27 1.27)) (justify left))
     )
-    (property "Footprint" "Resistor_SMD:R_0201_0603Metric" (at 159.512 77.47 90)
+    (property "Footprint" "Resistor_SMD:R_0402_1005Metric" (at 159.512 77.47 90)
       (effects (font (size 1.27 1.27)) hide)
     )
@@
       (effects (font (size 1.27 1.27)) hide)
     )
-    (property "LCSC" "C163490" (at 161.29 77.47 0)
+    (property "LCSC" "C25905" (at 161.29 77.47 0)
       (effects (font (size 1.27 1.27)) hide)
     )
-    (property "Basic/Extended" "E" (at 161.29 77.47 0)
+    (property "Basic/Extended" "B" (at 161.29 77.47 0)
       (effects (font (size 1.27 1.27)) hide)
     )
