File: hw/Watch/MainBoard.kicad_sch (KiCad schematic)
At the start: 8 parts, among them SW1 SW_Push

Commit message: wip
Parts:
- removed SW1: SW_Push, RLK-ElectorMechanicalComponents:TCF2QR, symbol Switch:SW_Push
Other:
- moved on the sheet: D13, R4, R5

Commit message: WIP
Parts:
- BZ1: footprint RKL-StandardPackages:PKLCS1212E-(RH-Logic_piezzo) -> RKL-Audio:SmallBuzzer; LCSC C113159 -> C255307
Changed lines of the file:
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@@
       (effects (font (size 1.27 1.27)))
     )
-    (property "Footprint" "RKL-StandardPackages:PKLCS1212E-(RH-Logic_piezzo)" (at 61.595 101.6 90)
+    (property "Footprint" "RKL-Audio:SmallBuzzer" (at 61.595 101.6 90)
       (effects (font (size 1.27 1.27)) hide)
     )
@@
       (effects (font (size 1.27 1.27)) hide)
     )
-    (property "LCSC" "C113159" (at 60.96 104.14 0)
+    (property "LCSC" "C255307" (at 60.96 104.14 0)
       (effects (font (size 1.27 1.27)) hide)
     )

Commit message: wip
Parts:
- removed D13: LED_Dual_AKAK, RKL-LED:SMD,1.5x3.2mm 4pin, symbol Device:LED_Dual_AKAK
- removed R1, R2, R3: 4.7k, Resistor_SMD:R_0402_1005Metric, symbol Device:R
- removed R4, R5: 1k, Resistor_SMD:R_0402_1005Metric, symbol Device:R
- added R7 (x3): 10k, Resistor_SMD:R_0201_0603Metric, symbol Device:R
Connections:
- net 3V3: now also R7.1, R7.1, R7.1
- net INT: now also R7.2
- net SCL: now also R7.2
- net SDA: now also R7.2
- no-connect marks 4 -> 21
Other:
- sheet ESP32-S3-MINI ports: added none; removed IO00-PU, IO03-FLOATING, IO45-PD, IO46-PD

Commit message: PCB
Parts:
- R7: footprint Resistor_SMD:R_0201_0603Metric -> Resistor_SMD:R_0402_1005Metric; Basic/Extended E -> B; LCSC C106225 -> C25744
Changed lines of the file:
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@@
       (effects (font (size 1.27 1.27)) (justify left))
     )
-    (property "Footprint" "Resistor_SMD:R_0201_0603Metric" (at 155.702 69.85 90)
+    (property "Footprint" "Resistor_SMD:R_0402_1005Metric" (at 155.702 69.85 90)
       (effects (font (size 1.27 1.27)) hide)
     )
@@
       (effects (font (size 1.27 1.27)) hide)
     )
-    (property "LCSC" "C106225" (at 157.48 69.85 0)
+    (property "LCSC" "C25744" (at 157.48 69.85 0)
       (effects (font (size 1.27 1.27)) hide)
     )
@@
       (effects (font (size 1.27 1.27)) hide)
     )
-    (property "Basic/Extended" "E" (at 157.48 69.85 0)
+    (property "Basic/Extended" "B" (at 157.48 69.85 0)
       (effects (font (size 1.27 1.27)) hide)
     )
@@
       (effects (font (size 1.27 1.27)) (justify left))
     )
-    (property "Footprint" "Resistor_SMD:R_0201_0603Metric" (at 163.322 69.85 90)
+    (property "Footprint" "Resistor_SMD:R_0402_1005Metric" (at 163.322 69.85 90)
       (effects (font (size 1.27 1.27)) hide)
     )
@@
       (effects (font (size 1.27 1.27)) hide)
     )
-    (property "LCSC" "C106225" (at 165.1 69.85 0)
+    (property "LCSC" "C25744" (at 165.1 69.85 0)
       (effects (font (size 1.27 1.27)) hide)
     )
@@
       (effects (font (size 1.27 1.27)) hide)
     )
-    (property "Basic/Extended" "E" (at 165.1 69.85 0)
+    (property "Basic/Extended" "B" (at 165.1 69.85 0)
       (effects (font (size 1.27 1.27)) hide)
     )
@@
       (effects (font (size 1.27 1.27)) (justify left))
     )
-    (property "Footprint" "Resistor_SMD:R_0201_0603Metric" (at 148.082 69.85 90)
+    (property "Footprint" "Resistor_SMD:R_0402_1005Metric" (at 148.082 69.85 90)
       (effects (font (size 1.27 1.27)) hide)
     )
@@
       (effects (font (size 1.27 1.27)) hide)
     )
-    (property "LCSC" "C106225" (at 149.86 69.85 0)
+    (property "LCSC" "C25744" (at 149.86 69.85 0)
       (effects (font (size 1.27 1.27)) hide)
     )
@@
       (effects (font (size 1.27 1.27)) hide)
     )
-    (property "Basic/Extended" "E" (at 149.86 69.85 0)
+    (property "Basic/Extended" "B" (at 149.86 69.85 0)
       (effects (font (size 1.27 1.27)) hide)
     )
@@
       (effects (font (size 1.27 1.27)) (justify right))
     )
-    (pin "IO04" bidirectional (at 139.7 76.2 0)
-      (effects (font (size 1.27 1.27)) (justify right))
-    )
-    (pin "IO06" bidirectional (at 139.7 82.55 0)
-      (effects (font (size 1.27 1.27)) (justify right))
-    )
+    (pin "IO04" bidirectional (at 139.7 82.55 0)
+      (effects (font (size 1.27 1.27)) (justify right))
+    )
+    (pin "IO06" bidirectional (at 139.7 76.2 0)
+      (effects (font (size 1.27 1.27)) (justify right))
+    )
